File: hodiny.brd (EAGLE design)
At the start: 147 x 54 mm, 101 parts, among them IC1 74HC42D, IC2 MC34063AD, IC3 UA78M33DCY, J1 12V, Q2 IRF740, Q3 MMBTA56-SOT23, T1 BTA42, T10 BTA42, T11 BTA42, T12 BTA42, T13 BTA42, T14 BTA92, T15 BTA42, T16 BTA92, T17 BTA42, T18 BTA92, T19 BTA42, T2 BTA92, T20 BTA92, T21 BTA42, T22 BTA92, T3 BTA42, T4 BTA42, T5 BTA42, T6 BTA42, T7 BTA42, T8 BTA42, T9 BTA42, U1 LPC812M101JD20, X1 SMCE-5032

Commit message: REV2 - Red Board
Parts:
- removed IC1: 74HC42D, 74xx-eu:SO16
- removed JP3: (no value), jumper:JP4
- removed JP4: (no value), jumper:JP1
- added D4, D5, D6, D7, D8, D9: BAV103, diode:MINIMELF
- added IC4: 4028D, 40xx:SO16
- added R38, R42: 47K, rcl:0207/7
- added R43, R44, R45, R46, R47, R48, R49, R50, R51, R52, R53: 220K, rcl:R1206
- added U$1: ESP8266-LIM, esp8266-lim:ESP8266-LIM
- C8, C9: value 18p -> 39p
- Q2: value IRF740 -> IRF740H; device transistor-power:TO220BV -> transistor-power:TO220BH
- R18: device rcl:RTRIMTSM53YJ -> rcl:RTRIM4G/J
- moved C12 24.7 mm to (31.4, 36.4), turned to 0 degrees
- moved D3 20.8 mm to (31.4, 28.3), turned to 270 degrees
- moved R17 14.3 mm to (23.1, 48.4), flipped to the bottom
- moved Q2 7.44 mm to (9.04, 30.7), turned to 0 degrees
- moved L2 4.48 mm to (21.4, 30.4), turned to 0 degrees
- moved D1 2.10 mm to (53.1, 33.3)
- moved R35 1.85 mm to (114.0, 24.9)
- moved R8 1.68 mm to (112.0, 34.9)
- moved R7 1.68 mm to (112.0, 32.7)
- moved R5 1.68 mm to (112.0, 28.4)
- moved R6 1.68 mm to (112.0, 30.5)
- moved R41 1.67 mm to (22.9, 22.1)
- moved R36 1.59 mm to (111.7, 24.9)
- moved T21 1.20 mm to (108.7, 25.1)
- moved R18 1.03 mm to (12.6, 48.4), turned to 270 degrees
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Connections:
- removed net N$9: JP3.2, U1.18
- removed net V+: C12.+, D3.C, JP4.1, R1.2, R17.1, R19.2, R23.2, R27.2, R31.2, R35.2, T14.E, T16.E, T18.E, T2.E, T20.E, T22.E
- new net 100V: D4.A, D5.A, D6.A, D7.A, D8.A, D9.A, R38.2, R42.1, R43.2, R44.2, R45.2, R46.2, R47.2, R48.2, R49.2, R50.2, R51.2, R52.2, R53.2
- new net 180V: C12.+, D3.C, R1.2, R17.1, R19.2, R23.2, R27.2, R31.2, R35.2, R38.1, T14.E, T16.E, T18.E, T2.E, T20.E, T22.E
- new net K10: N1.10, N1.4, N2.10, N2.4, N3.10, N3.4, N4.10, N4.4, N5.10, N5.4, N6.10, N6.4, R48.1
- new net N$68: U$1.TX, U1.19
- net +3V3: now also IC4.16, U$1.3V3; no longer IC1.16, JP3.1
- net BCD_A: now also IC4.10, U1.5; no longer IC1.15, U1.10
- net BCD_B: now also IC4.13, U1.10; no longer IC1.14, R39.2, U1.9
- net BCD_C: now also IC4.12, R39.2, U1.9; no longer IC1.13, R40.2, U1.8
- net BCD_D: now also IC4.11, R40.2, U1.8; no longer IC1.12, U1.5
- net GND: now also IC4.8, R42.2, U$1.GND; no longer IC1.8, JP3.4, JP4.2
- net K0: now also R47.1, T5.C; no longer T4.C
- net K1: now also R46.1, T11.C; no longer T3.C
- net K2: now also R43.1, T3.C; no longer T5.C
- net K3: now also R45.1, T12.C; no longer T6.C
- net K4: now also R44.1, T4.C; no longer T7.C
- net K5: now also R49.1
- net K6: now also R50.1
- net K7: now also R51.1, T6.C; no longer T10.C
- net K8: now also R52.1, T10.C; no longer T11.C
- net K9: now also R53.1, T7.C; no longer T12.C
- net N$10: now also U$1.RX, U1.18; no longer JP3.3, U1.19
- net N$18: now also IC4.1; no longer IC1.1
- net N$19: now also D5.C
- net N$20: now also IC4.2; no longer IC1.2
- net N$21: now also IC4.3; no longer IC1.3
- net N$22: now also IC4.4; no longer IC1.4
- net N$23: now also IC4.5; no longer IC1.5
- net N$24: now also IC4.6; no longer IC1.6
- net N$25: now also IC4.7; no longer IC1.7
- net N$26: now also IC4.9; no longer IC1.9
- net N$27: now also IC4.14; no longer IC1.10
- net N$28: now also IC4.15; no longer IC1.11
- net N$49: now also D4.C
- net N$55: now also D6.C
- net N$61: now also D7.C
- net N$67: now also D8.C
- net N$73: now also D9.C
Routing:
- net 100V: track 0.00 -> 194.6 mm
- net V+: track 176.7 -> 0.00 mm
- net 180V: track 0.00 -> 154.5 mm
- net K10: track 0.00 -> 137.7 mm
- net N$68: track 0.00 -> 69.7 mm, vias 0 -> 1
- net N$10: track 15.1 -> 71.0 mm, vias 0 -> 1
- net K1: track 144.3 -> 192.3 mm, vias 1 -> 2
- net K7: track 221.9 -> 187.4 mm
- net K8: track 212.7 -> 239.3 mm, vias 1 -> 5
- net K3: track 169.9 -> 191.4 mm, vias 1 -> 0
- net K0: track 146.1 -> 165.8 mm
- net +3V3: track 71.6 -> 90.7 mm, vias 0 -> 1
- net N$41: track 12.3 -> 26.0 mm
- net N$9: track 12.5 -> 0.00 mm
- net K9: track 208.9 -> 197.0 mm, vias 1 -> 2
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Other:
- board text added: "Ondrej Kosta 2017 REV2"
- board text removed: "Ondrej Kosta 2016"
