File: hodiny.sch (EAGLE design)
At the start: 101 parts, among them IC1 74HC42D, IC2 MC34063AD, IC3 UA78M33DCY, J1 12V, Q2 IRF740, Q3 MMBTA56-SOT23, T1 BTA42, T10 BTA42, T11 BTA42, T12 BTA42, T13 BTA42, T14 BTA92, T15 BTA42, T16 BTA92, T17 BTA42, T18 BTA92, T19 BTA42, T2 BTA92, T20 BTA92, T21 BTA42, T22 BTA92, T3 BTA42, T4 BTA42, T5 BTA42, T6 BTA42, T7 BTA42, T8 BTA42, T9 BTA42, U1 LPC812M101JD20, X1 SMCE-5032

Commit message: REV2 - Red Board
Parts:
- removed IC1: 74HC42D, 74xx-eu:74HC42D
- removed JP3: (no value), jumper:JP4E
- removed JP4: (no value), jumper:JP1E
- added D4, D5, D6, D7, D8, D9: BAV103, diode:DIODE-MINIMELF
- added IC4: 4028D, 40xx:4028D
- added R38, R42: 47K, rcl:R-EU_0207/7
- added R43, R44, R45, R46, R47, R48, R49, R50, R51, R52, R53: 220K, rcl:R-EU_R1206
- added U$1: ESP8266-LIM, esp8266-lim:ESP8266-LIM
- C8, C9: value 18p -> 39p
- Q2: value IRF740 -> IRF740H; device transistor-power:IRF740 -> transistor-power:IRF740H
- R18: device rcl:R-TRIMMTSM53YJ -> rcl:R-TRIMM4G/J
Connections:
- removed net N$9: JP3.2, U1.PIO0_6/VDDCMP
- removed net V+: C12.+, D3.C, JP4.1, R1.2, R17.1, R19.2, R23.2, R27.2, R31.2, R35.2, T14.E, T16.E, T18.E, T2.E, T20.E, T22.E
- new net 100V: D4.A, D5.A, D6.A, D7.A, D8.A, D9.A, R38.2, R42.1, R43.2, R44.2, R45.2, R46.2, R47.2, R48.2, R49.2, R50.2, R51.2, R52.2, R53.2
- new net 180V: C12.+, D3.C, R1.2, R17.1, R19.2, R23.2, R27.2, R31.2, R35.2, R38.1, T14.E, T16.E, T18.E, T2.E, T20.E, T22.E
- new net K10: N1.DP, N1.IC, N2.DP, N2.IC, N3.DP, N3.IC, N4.DP, N4.IC, N5.DP, N5.IC, N6.DP, N6.IC, R48.1
- new net N$68: U$1.TX, U1.PIO0_0/ACMP_I1/TDO
- net +3V3: now also IC4P.VDD, U$1.3V3; no longer IC1P.VCC, JP3.1
- net BCD_A: now also IC4A.A, U1.PIO0_4/WAKEUP/!TRST!; no longer IC1A.A, U1.PIO0_16
- net BCD_B: now also IC4A.B, U1.PIO0_16; no longer IC1A.B, R39.2, U1.PIO0_10
- net BCD_C: now also IC4A.C, R39.2, U1.PIO0_10; no longer IC1A.C, R40.2, U1.PIO0_11
- net BCD_D: now also IC4A.D, R40.2, U1.PIO0_11; no longer IC1A.D, U1.PIO0_4/WAKEUP/!TRST!
- net GND: now also IC4P.VSS, R42.2, U$1.GND; no longer IC1P.GND, JP3.4, JP4.2
- net K0: now also R47.1, T5.C; no longer T4.C
- net K1: now also R46.1, T11.C; no longer T3.C
- net K2: now also R43.1, T3.C; no longer T5.C
- net K3: now also R45.1, T12.C; no longer T6.C
- net K4: now also R44.1, T4.C; no longer T7.C
- net K5: now also R49.1
- net K6: now also R50.1
- net K7: now also R51.1, T6.C; no longer T10.C
- net K8: now also R52.1, T10.C; no longer T11.C
- net K9: now also R53.1, T7.C; no longer T12.C
- net N$10: now also U$1.RX, U1.PIO0_6/VDDCMP; no longer JP3.3, U1.PIO0_0/ACMP_I1/TDO
- net N$18: now also IC4A.Q4; no longer IC1A.O0
- net N$19: now also D5.C
- net N$20: now also IC4A.Q2; no longer IC1A.O1
- net N$21: now also IC4A.Q0; no longer IC1A.O2
- net N$22: now also IC4A.Q7; no longer IC1A.O3
- net N$23: now also IC4A.Q9; no longer IC1A.O4
- net N$24: now also IC4A.Q5; no longer IC1A.O5
- net N$25: now also IC4A.Q6; no longer IC1A.O6
- net N$26: now also IC4A.Q8; no longer IC1A.O7
- net N$27: now also IC4A.Q1; no longer IC1A.O8
- net N$28: now also IC4A.Q3; no longer IC1A.O9
- net N$49: now also D4.C
- net N$55: now also D6.C
- net N$61: now also D7.C
- net N$67: now also D8.C
- net N$73: now also D9.C
Other:
- moved on the sheet: R1, R10, R11, R12, R13, R14, R19, R2, R20, R21, R22, R23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
